Commit message: Modified the arm's and gripper's description files to rectify some issues

File: kortex_description/gen3_arm/urdf/gen3_macro.xacro (robot description, xacro)
@@ -5,43 +5,25 @@
   <xacro:property name="PI" value="3.1415926535897931"/>
   <xacro:macro name="load_arm" params="
-    parent
-    dof
-    vision
+    parent:=world
+    vision:=false
     prefix
     *origin
-    robot_ip
+    robot_ip:=192.168.1.10
     username:=admin
     password:=admin
     port:=10000
     port_realtime:=10001
-    session_inactivity_timeout_ms:=6000
+    session_inactivity_timeout_ms:=60000
     connection_inactivity_timeout_ms:=2000
-    use_internal_bus_gripper_comm:=true
-    gripper_joint_name
-    gripper_max_velocity:=100.0
-    gripper_max_force:=100.0
-    use_fake_hardware:=false
-    fake_sensor_commands:=false
-    sim_gazebo:=false
-    sim_ignition:=false
-    sim_isaac:=false
-    isaac_joint_commands:=/isaac_joint_commands
-    isaac_joint_states:=/isaac_joint_states
-    use_external_cable:=false
-    initial_positions:=${dict(joint_1=0.0,joint_2=0.0,joint_3=0.0,joint_4=0.0,joint_5=0.0,joint_6=0.0,joint_7=0.0)}
-    moveit_active:=false">
+    use_internal_bus_gripper_comm:=false
+    tf_prefix
+    gripper_joint_name:=finger_joint
+    gripper_max_velocity:=100
+    gripper_max_force:=100
+    use_external_cable:=false">
     <!-- ros2 control include -->
-    <xacro:include filename="$(find kortex_description)/arms/gen3/${dof}dof/urdf/kortex.ros2_control.xacro" />
+    <xacro:include filename="$(find kortex_description)/gen3_arm/urdf/kortex.ros2_control.xacro" />
     <xacro:kortex_ros2_control
       name="${prefix}KortexMultiInterfaceHardware" prefix="${prefix}"
-      use_fake_hardware="${use_fake_hardware}"
-      fake_sensor_commands="${fake_sensor_commands}"
-      sim_gazebo="${sim_gazebo}"
-      sim_ignition="${sim_ignition}"
-      sim_isaac="${sim_isaac}"
-      isaac_joint_commands="${isaac_joint_commands}"
-      isaac_joint_states="${isaac_joint_states}"
-      tf_prefix=""
-      initial_positions="${initial_positions}"
       robot_ip="${robot_ip}"
       username="${username}"
@@ -52,4 +34,5 @@
       connection_inactivity_timeout_ms="${connection_inactivity_timeout_ms}"
       use_internal_bus_gripper_comm="${use_internal_bus_gripper_comm}"
+      tf_prefix="${tf_prefix}"
       gripper_max_velocity="${gripper_max_velocity}"
       gripper_max_force="${gripper_max_force}"
@@ -69,14 +52,14 @@
         <origin xyz="0 0 0" rpy="0 0 0" />
         <geometry>
-          <mesh filename="file://$(find kortex_description)/arms/gen3/${dof}dof/meshes/base_link.dae" />
-        </geometry>
-        <material name="">
-          <color rgba="0.75294 0.75294 0.75294 1" />
-        </material>
-      </visual>
-      <collision>
-        <origin xyz="0 0 0" rpy="0 0 0" />
-        <geometry>
-          <mesh filename="file://$(find kortex_description)/arms/gen3/${dof}dof/meshes/base_link.dae" />
+          <mesh filename="file://$(find kortex_description)/gen3_arm/meshes/base_link.dae" />
+        </geometry>
+        <material name="">
+          <color rgba="0.75294 0.75294 0.75294 1" />
+        </material>
+      </visual>
+      <collision>
+        <origin xyz="0 0 0" rpy="0 0 0" />
+        <geometry>
+          <mesh filename="file://$(find kortex_description)/gen3_arm/meshes/base_link.dae" />
         </geometry>
       </collision>
@@ -91,14 +74,14 @@
         <origin xyz="0 0 0" rpy="0 0 0" />
         <geometry>
-          <mesh filename="file://$(find kortex_description)/arms/gen3/${dof}dof/meshes/shoulder_link.dae" />
-        </geometry>
-        <material name="">
-          <color rgba="0.75294 0.75294 0.75294 1" />
-        </material>
-      </visual>
-      <collision>
-        <origin xyz="0 0 0" rpy="0 0 0" />
-        <geometry>
-          <mesh filename="file://$(find kortex_description)/arms/gen3/${dof}dof/meshes/shoulder_link.dae" />
+          <mesh filename="file://$(find kortex_description)/gen3_arm/meshes/shoulder_link.dae" />
+        </geometry>
+        <material name="">
+          <color rgba="0.75294 0.75294 0.75294 1" />
+        </material>
+      </visual>
+      <collision>
+        <origin xyz="0 0 0" rpy="0 0 0" />
+        <geometry>
+          <mesh filename="file://$(find kortex_description)/gen3_arm/meshes/shoulder_link.dae" />
         </geometry>
       </collision>
@@ -147,14 +130,14 @@
         <origin xyz="0 0 0" rpy="0 0 0" />
         <geometry>
-          <mesh filename="file://$(find kortex_description)/arms/gen3/${dof}dof/meshes/half_arm_1_link.dae" />
-        </geometry>
-        <material name="">
-          <color rgba="0.75294 0.75294 0.75294 1" />
-        </material>
-      </visual>
-      <collision>
-        <origin xyz="0 0 0" rpy="0 0 0" />
-        <geometry>
-          <mesh filename="file://$(find kortex_description)/arms/gen3/${dof}dof/meshes/half_arm_1_link.dae" />
+          <mesh filename="file://$(find kortex_description)/gen3_arm/meshes/half_arm_1_link.dae" />
+        </geometry>
+        <material name="">
+          <color rgba="0.75294 0.75294 0.75294 1" />
+        </material>
+      </visual>
+      <collision>
+        <origin xyz="0 0 0" rpy="0 0 0" />
+        <geometry>
+          <mesh filename="file://$(find kortex_description)/gen3_arm/meshes/half_arm_1_link.dae" />
         </geometry>
       </collision>
@@ -181,14 +164,14 @@
         <origin xyz="0 0 0" rpy="0 0 0" />
         <geometry>
-          <mesh filename="file://$(find kortex_description)/arms/gen3/${dof}dof/meshes/half_arm_2_link.dae" />
-        </geometry>
-        <material name="">
-          <color rgba="0.75294 0.75294 0.75294 1" />
-        </material>
-      </visual>
-      <collision>
-        <origin xyz="0 0 0" rpy="0 0 0" />
-        <geometry>
-          <mesh filename="file://$(find kortex_description)/arms/gen3/${dof}dof/meshes/half_arm_2_link.dae" />
+          <mesh filename="file://$(find kortex_description)/gen3_arm/meshes/half_arm_2_link.dae" />
+        </geometry>
+        <material name="">
+          <color rgba="0.75294 0.75294 0.75294 1" />
+        </material>
+      </visual>
+      <collision>
+        <origin xyz="0 0 0" rpy="0 0 0" />
+        <geometry>
+          <mesh filename="file://$(find kortex_description)/gen3_arm/meshes/half_arm_2_link.dae" />
         </geometry>
       </collision>
@@ -237,14 +220,14 @@
         <origin xyz="0 0 0" rpy="0 0 0" />
         <geometry>
-          <mesh filename="file://$(find kortex_description)/arms/gen3/${dof}dof/meshes/forearm_link.dae" />
-        </geometry>
-        <material name="">
-          <color rgba="0.75294 0.75294 0.75294 1" />
-        </material>
-      </visual>
-      <collision>
-        <origin xyz="0 0 0" rpy="0 0 0" />
-        <geometry>
-          <mesh filename="file://$(find kortex_description)/arms/gen3/${dof}dof/meshes/forearm_link.dae" />
+          <mesh filename="file://$(find kortex_description)/gen3_arm/meshes/forearm_link.dae" />
+        </geometry>
+        <material name="">
+          <color rgba="0.75294 0.75294 0.75294 1" />
+        </material>
+      </visual>
+      <collision>
+        <origin xyz="0 0 0" rpy="0 0 0" />
+        <geometry>
+          <mesh filename="file://$(find kortex_description)/gen3_arm/meshes/forearm_link.dae" />
         </geometry>
       </collision>
@@ -271,14 +254,14 @@
         <origin xyz="0 0 0" rpy="0 0 0" />
         <geometry>
-          <mesh filename="file://$(find kortex_description)/arms/gen3/${dof}dof/meshes/spherical_wrist_1_link.dae" />
-        </geometry>
-        <material name="">
-          <color rgba="0.75294 0.75294 0.75294 1" />
-        </material>
-      </visual>
-      <collision>
-        <origin xyz="0 0 0" rpy="0 0 0" />
-        <geometry>
-          <mesh filename="file://$(find kortex_description)/arms/gen3/${dof}dof/meshes/spherical_wrist_1_link.dae" />
+          <mesh filename="file://$(find kortex_description)/gen3_arm/meshes/spherical_wrist_1_link.dae" />
+        </geometry>
+        <material name="">
+          <color rgba="0.75294 0.75294 0.75294 1" />
+        </material>
+      </visual>
+      <collision>
+        <origin xyz="0 0 0" rpy="0 0 0" />
+        <geometry>
+          <mesh filename="file://$(find kortex_description)/gen3_arm/meshes/spherical_wrist_1_link.dae" />
         </geometry>
       </collision>
@@ -327,14 +310,14 @@
         <origin xyz="0 0 0" rpy="0 0 0" />
         <geometry>
-          <mesh filename="file://$(find kortex_description)/arms/gen3/${dof}dof/meshes/spherical_wrist_2_link.dae" />
-        </geometry>
-        <material name="">
-          <color rgba="0.75294 0.75294 0.75294 1" />
-        </material>
-      </visual>
-      <collision>
-        <origin xyz="0 0 0" rpy="0 0 0" />
-        <geometry>
-          <mesh filename="file://$(find kortex_description)/arms/gen3/${dof}dof/meshes/spherical_wrist_2_link.dae" />
+          <mesh filename="file://$(find kortex_description)/gen3_arm/meshes/spherical_wrist_2_link.dae" />
+        </geometry>
+        <material name="">
+          <color rgba="0.75294 0.75294 0.75294 1" />
+        </material>
+      </visual>
+      <collision>
+        <origin xyz="0 0 0" rpy="0 0 0" />
+        <geometry>
+          <mesh filename="file://$(find kortex_description)/gen3_arm/meshes/spherical_wrist_2_link.dae" />
         </geometry>
       </collision>
@@ -362,14 +345,14 @@
         <origin xyz="0 0 0" rpy="0 0 0" />
         <geometry>
-          <mesh filename="file://$(find kortex_description)/arms/gen3/${dof}dof/meshes/bracelet_with_vision_link.dae" />
-        </geometry>
-        <material name="">
-          <color rgba="0.75294 0.75294 0.75294 1" />
-        </material>
-      </visual>
-      <collision>
-        <origin xyz="0 0 0" rpy="0 0 0" />
-        <geometry>
-          <mesh filename="file://$(find kortex_description)/arms/gen3/${dof}dof/meshes/bracelet_with_vision_link.dae" />
+          <mesh filename="file://$(find kortex_description)/gen3_arm/meshes/bracelet_with_vision_link.dae" />
+        </geometry>
+        <material name="">
+          <color rgba="0.75294 0.75294 0.75294 1" />
+        </material>
+      </visual>
+      <collision>
+        <origin xyz="0 0 0" rpy="0 0 0" />
+        <geometry>
+          <mesh filename="file://$(find kortex_description)/gen3_arm/meshes/bracelet_with_vision_link.dae" />
         </geometry>
       </collision>
@@ -386,14 +369,14 @@
         <origin xyz="0 0 0" rpy="0 0 0" />
         <geometry>
-          <mesh filename="file://$(find kortex_description)/arms/gen3/${dof}dof/meshes/bracelet_no_vision_link.dae" />
-        </geometry>
-        <material name="">
-          <color rgba="0.75294 0.75294 0.75294 1" />
-        </material>
-      </visual>
-      <collision>
-        <origin xyz="0 0 0" rpy="0 0 0" />
-        <geometry>
-          <mesh filename="file://$(find kortex_description)/arms/gen3/${dof}dof/meshes/bracelet_no_vision_link.dae" />
+          <mesh filename="file://$(find kortex_description)/gen3_arm/meshes/bracelet_no_vision_link.dae" />
+        </geometry>
+        <material name="">
+          <color rgba="0.75294 0.75294 0.75294 1" />
+        </material>
+      </visual>
+      <collision>
+        <origin xyz="0 0 0" rpy="0 0 0" />
+        <geometry>
+          <mesh filename="file://$(find kortex_description)/gen3_arm/meshes/bracelet_no_vision_link.dae" />
         </geometry>
       </collision>
@@ -447,26 +430,4 @@
     </joint>
     <xacro:if value="${vision}">
-      <!-- sim camera needs to be rotated which might not apply to built in vision module -->
-      <xacro:if value="${sim_ignition}">
-        <link name="${prefix}camera_link" />
-        <joint name="${prefix}camera_module" type="fixed">
-          <origin xyz="0 0.05639 0.01305" rpy="0 ${-PI/2} ${-PI/2}" />
-          <parent link="${prefix}end_effector_link" />
-          <child  link="${prefix}camera_link" />
-        </joint>
-        <link name="${prefix}camera_depth_frame" />
-        <joint name="${prefix}depth_module" type="fixed">
-          <origin xyz="0.0275 0.066 0.01305" rpy="0 ${-PI/2} ${-PI/2}" />
-          <parent link="${prefix}end_effector_link" />
-          <child  link="${prefix}camera_depth_frame" />
-        </joint>
-        <link name="${prefix}camera_color_frame" />
-        <joint name="${prefix}color_module" type="fixed">
-          <origin xyz="0 0.05639 0.01305" rpy="0 ${-PI/2} ${-PI/2}" />
-          <parent link="${prefix}end_effector_link" />
-          <child  link="${prefix}camera_color_frame" />
-        </joint>
-      </xacro:if>
-      <xacro:unless value="${sim_ignition}">
         <link name="${prefix}camera_link" />
         <joint name="${prefix}camera_module" type="fixed">
@@ -487,5 +448,4 @@
           <child  link="${prefix}camera_color_frame" />
         </joint>
-      </xacro:unless>
     </xacro:if>
   </xacro:macro>

File: kortex_description/gripper_robotiq_2f_85/urdf/robotiq_2f_85_macro.xacro (robot description, xacro)
@@ -2,19 +2,14 @@
 <robot name="robotiq_2f_85_model" xmlns:xacro="http://ros.org/wiki/xacro">
   <xacro:macro name="load_gripper" params="
-    parent
+    parent:=end_effector_link
     prefix
-    use_fake_hardware:=false
-    fake_sensor_commands:=false
-    sim_ignition:=false
-    sim_isaac:=false
-    isaac_joint_commands:=/isaac_joint_commands
-    isaac_joint_states:=/isaac_joint_states
     use_internal_bus_gripper_comm:=false
-    com_port:=/dev/ttyUSB0
-    moveit_active:=false">
+    com_port:=/dev/ttyUSB0">
     <xacro:include filename="$(find robotiq_description)/urdf/robotiq_2f_85_macro.urdf.xacro" />
     <!-- Hardware talks directly to the gripper so we don't need ros2_control unless we are simulating -->
-    <xacro:property name="include_ros2_control" value="false"/>
-    <xacro:if value="${sim_ignition or sim_isaac or use_fake_hardware or not use_internal_bus_gripper_comm}">
+    <xacro:if value="${use_internal_bus_gripper_comm}">
+      <xacro:property name="include_ros2_control" value="false"/>
+    </xacro:if>
+    <xacro:if value="${not use_internal_bus_gripper_comm}">
       <xacro:property name="include_ros2_control" value="true"/>
     </xacro:if>
@@ -24,11 +19,5 @@
         parent="${parent}"
         include_ros2_control="${include_ros2_control}"
-        com_port="${com_port}"
-        use_fake_hardware="${use_fake_hardware}"
-        fake_sensor_commands="${fake_sensor_commands}"
-        sim_ignition="${sim_ignition}"
-        sim_isaac="${sim_isaac}"
-        isaac_joint_commands="${isaac_joint_commands}"
-        isaac_joint_states="${isaac_joint_states}">
+        com_port="${com_port}">
         <origin xyz="0 0 0" rpy="0 0 0" />
     </xacro:robotiq_gripper>
